File: project/ZSWatch.kicad_sch (KiCad schematic)
At the start: 72 parts, among them IC1 APDS-9306-065, IC10 FAN5622SX, IC11 XC9265A331MR-G, IC12 BMP581, IC13 BME688, IC14 LIS2MDLTR, IC15 DRV2603RUNT, IC2 ESDALC6V1W5, IC3 MAX1811ESA+, IC4 DMC2400UV-7, IC5 NCV300LSN36T1G, IC6 AT25SL128A, IC7 XC9265C181MR-G, IC8 BMI270, IC9 NTS0104GU12, M1 NORA-B106, M2 Vibrator DC Motor, X1 DOCK, X10 M-, X2 BATTERY, X3 GPIO0, X4 GPIO1, X5 GPIO2, X6 GPIO3, X7 GND, X8 GC9A01A_CST816S, X9 M+

Commit message: Initialize branch
Parts:
- removed C1, C10, C13, C15, C17, C19, C20, C21, C7, C8, C9: 100n, Capacitor_SMD:C_0603_1608Metric, symbol Device:C_Small
- removed C11, C18, C4: 10u, Capacitor_SMD:C_0603_1608Metric, symbol Device:C_Small
- removed C12: 1u, Capacitor_SMD:C_0603_1608Metric, symbol Device:C_Small
- removed C14, C6: 22u, Capacitor_SMD:C_0603_1608Metric, symbol Device:C_Small
- removed C16: 220n, Capacitor_SMD:C_0603_1608Metric, symbol Device:C_Small
- removed C3: 2u2, Capacitor_SMD:C_0603_1608Metric, symbol Device:C_Small
- removed IC1: APDS-9306-065, OptoDevice:Broadcom_DFN-6_2x2mm_P0.65mm, symbol Sensor_Optical:APDS-9306-065
- removed IC10: FAN5622SX, Package_TO_SOT_SMD:TSOT-23-6, symbol ON Semiconductor:FAN5622SX
- removed IC11: XC9265A331MR-G, Package_SOT_SMD:SOT-25-5, symbol Torex Seimoconductor:XC9265A331MR-G
- removed IC12: BMP581, Package_LGA_Kampi:Bosch_LGA-10_2x2mm_P0.5mm_ClockwisePinNumbering, symbol Bosch_Kampi:BMP581
- removed IC13: BME688, Package_LGA_Kampi:Bosch_LGA-8_3x3mm_P0.8mm_ClockwisePinNumbering, symbol Bosch_Kampi:BME688
- removed IC14: LIS2MDLTR, Package_LGA_Kampi:LGA-12_2x2mm_P0.5mm, symbol ST:LIS2MDLTR
- removed IC15: DRV2603RUNT, Package_QFN:WQFN-10_2x2mm_P0.5mm, symbol TexasInstruments_Kampi:DRV2603RUNT
- removed IC2: ESDALC6V1W5, Package_SOT_SMD:SOT-325-5, symbol ST:ESDALC6V1W5
- removed IC3: MAX1811ESA+, Package_SO:SOIC-8_3.9x4.9mm_P1.27mm, symbol Battery_Management:MAX1811
- removed IC4: DMC2400UV-7, Package_TO_SOT_SMD:SOT-563, symbol Diodes Incorporated:DMC2400UV-7
- removed IC5: NCV300LSN36T1G, Package_SO:TSOP-5_1.65x3.05mm_P0.95mm, symbol ON Semiconductor:NCV300LSN36T1G
- removed IC7: XC9265C181MR-G, Package_SOT_SMD:SOT-25-5, symbol Torex Seimoconductor:XC9265C181MR-G
- removed IC8: BMI270, Package_LGA_Kampi:LGA-14_3x2.5mm_P0.5mm_LayoutBorder3x4y, symbol Bosch_Kampi:BMI270
- removed IC9: NTS0104GU12, Package_QFN:XQFN-12-1.7x2mm_P0.4mm, symbol NXP:NTS0104GU12
- removed L1, L2: 10u, Inductor_SMD:L_0603_1608Metric, symbol Device:L_Small
- removed M2: Vibrator DC Motor, symbol Motor:Motor_DC
- removed R1, R5: 1M, Resistor_SMD:R_0603_1608Metric, symbol Device:R_Small
- removed R11, R9: 100k, Resistor_SMD:R_0603_1608Metric, symbol Device:R_Small
- removed R12: 10k, Resistor_SMD:R_0603_1608Metric, symbol Device:R_Small
- removed R2: 1M5 / 0.1%, Resistor_SMD:R_0603_1608Metric, symbol Device:R_Small
- removed R3: 220k / 0.1%, Resistor_SMD:R_0603_1608Metric, symbol Device:R_Small
- removed R7, R8: 4k7, Resistor_SMD:R_0603_1608Metric, symbol Device:R_Small
- removed S1, S2, S3, S4: TL6340AF160Q, E-Switch:TL6340AF160Q_Modified, symbol Switch:SW_Push
- removed TP1: RESET, TestPoint:TestPoint_Pad_D1.0mm, symbol Connector:TestPoint
- removed TP2: SCL, TestPoint:TestPoint_Pad_D1.0mm, symbol Connector:TestPoint
- removed TP3: SDA, TestPoint:TestPoint_Pad_D1.0mm, symbol Connector:TestPoint
- removed TP4: 3V3, TestPoint:TestPoint_Pad_D1.0mm, symbol Connector:TestPoint
- removed TP5: BAT, TestPoint:TestPoint_Pad_D1.0mm, symbol Connector:TestPoint
- removed TP6: 1V8, TestPoint:TestPoint_Pad_D1.0mm, symbol Connector:TestPoint
- removed X10: M-, TestPoint:TestPoint_Pad_1.0x1.0mm, symbol Connector_Generic:Conn_01x01
- removed X2: BATTERY, Molex:2121340002, symbol Connector_Generic:Conn_01x02
- removed X3: GPIO0, TestPoint:TestPoint_Pad_1.0x1.0mm, symbol Connector_Generic:Conn_01x01
- removed X4: GPIO1, TestPoint:TestPoint_Pad_1.0x1.0mm, symbol Connector_Generic:Conn_01x01
- removed X5: GPIO2, TestPoint:TestPoint_Pad_1.0x1.0mm, symbol Connector_Generic:Conn_01x01
- removed X6: GPIO3, TestPoint:TestPoint_Pad_1.0x1.0mm, symbol Connector_Generic:Conn_01x01
- removed X7: GND, TestPoint:TestPoint_Pad_1.0x1.0mm, symbol Connector_Generic:Conn_01x01
- removed X8: GC9A01A_CST816S, EastRising:ER-CON0.4-24P, symbol Display:GC9A01A_CST816S
- removed X9: M+, TestPoint:TestPoint_Pad_1.0x1.0mm, symbol Connector_Generic:Conn_01x01
- added IC2: NX3DV42, symbol NXP:NX3DV42
- added R4: 100k, Resistor_SMD:R_0603_1608Metric, symbol Device:R_Small
- added X1: Conn_01x02, Connector_PinHeader_2.54mm:PinHeader_1x02_P2.54mm_Vertical, symbol Connector_Generic:Conn_01x02
- C2: value 4u7 -> 100n; Mfr. No. 06036D475KAT2A -> 06035C104KAT2A; Order Number 581-06036D475K -> 581-06035C104KAT2A
- IC1: renamed from IC6; Mfr. No. AT25SL128A -> AT25SL128A-MHE-T
- renumbered C5 to C1, R4 to R1, R6 to R2, R10 to R3, X1 to X2
Connections:
- net +1V8: now also X1.1 (Pin_1)
- net GND: now also IC2.3 (GND), IC2.8 (~{OE}), X1.2 (Pin_2)
- net VBUS: now also M1.B9 (VBUS), IC2.9 (Vcc), R4.1
- net MCU-D+: now reaches M1.C9 (D+)
- net MCU_D-: now reaches M1.D9 (D-)
- net MCU_D-: now also IC2.6 (HSD2-)
- net BAT_MON: no longer names the net of M1.J8 (P0.28/AIN7)
- net BAT_MON_EN: no longer names the net of M1.J7 (P1.10)
- net BMP581_INT: no longer names the net of M1.G3 (P0.25/AIN4)
- net BTN_1: no longer names the net of M1.H3 (P0.27/AIN6)
- net BTN_2: no longer names the net of M1.H8 (P0.30)
- net BTN_3: no longer names the net of M1.G8 (P1.12)
- net BTN_4: no longer names the net of M1.G1 (P1.06)
- net CHG: no longer names the net of M1.G9 (P1.13)
- net DISPLAY_BLK: no longer names the net of M1.D7 (P0.23)
- net DISPLAY_CLK: no longer names the net of M1.B1 (P0.08/TRACEDATA[3])
- net DISPLAY_CS: no longer names the net of M1.B3 (P0.11/TRACEDATA[0])
- net DISPLAY_DATA: no longer names the net of M1.C2 (P0.09/TRACEDATA[2])
- net DISPLAY_DC: no longer names the net of M1.A2 (P0.12/TRACECLK)
- net DISPLAY_EN: no longer names the net of M1.D1 (P0.15/QSPI[2])
- net DISPLAY_RST: no longer names the net of M1.B5 (P0.03/NFC2)
- net DRV_VIB_EN: no longer names the net of M1.F8 (P1.14)
- net DRV_VIB_PWM: no longer names the net of M1.F9 (P1.15)
- net GPIO0: no longer names the net of M1.C8 (P0.22)
- net GPIO1: no longer names the net of M1.D8 (P0.04/AIN0)
- net GPIO2: no longer names the net of M1.E8 (P0.05/AIN1)
- net GPIO3: no longer names the net of M1.E9 (P1.05)
- net INT1_LIS: no longer names the net of M1.E3 (P0.21)
- net INT2_LIS: no longer names the net of M1.E2 (P0.14/QSPI[1])
- net LIS2MDL_INT: no longer names the net of M1.H1 (P0.24)
- net RESETn renamed MCU_RESETn
- net MCU_RESETn: no longer X2.3 (Pin_3)
- net SENSOR_SCL: no longer names the net of M1.E1 (P0.18/QSPI_CS)
- net SENSOR_SDA: no longer names the net of M1.F1 (P0.17/QSPI_CLK)
- net SWDCLK renamed D+/SWDCLK
- net D+/SWDCLK: now also IC2.1 (D+); no longer M1.J2 (SWDCLK)
- net SWDIO renamed D-/SWDIO
- net D-/SWDIO: now also IC2.2 (D-); no longer M1.H2 (SWDIO)
- net TOUCH_INT: no longer names the net of M1.A4 (P1.00)
- net TOUCH_RST: no longer names the net of M1.A5 (P0.20)
- net TOUCH_SCL: no longer names the net of M1.A3 (P1.03/I2C)
- net TOUCH_SDA: no longer names the net of M1.B4 (P1.02/I2C)
- new net MCU_D+: IC2.7 (HSDI2+)
- new net MCU_SWDCLK: IC2.5 (HSDI1+), M1.J2 (SWDCLK)
- new net MCU_SWDIO: IC2.4 (HSD1-), M1.H2 (SWDIO)
- new net SEL_SWD: IC2.10 (S), R4.2, X2.3 (Pin_3)
- no-connect marks 30 -> 49
Other:
- note added: "S Channel Function L HSD1+ and HSD1- SWD H HSD2+ and HSD2- USB (Default)"
- note removed: "1.8<->3.3 level shifter"
- note removed: "1V8 regulator"
- note removed: "9.53k gives I_{LED} 30mA (max)"
- note removed: "Battery can do 500mA charging however it requires the source to deliver 500mA. USB hubs for example may only deliver 100mA. Not sure what will happen in that case if set charger to 500mA. Stay safe and use 100mA for now."
- note removed: "Battery supervisor"
- note removed: "Buttons"
- note removed: "CHG is open-drain so open with internal pullup enabled"
- note removed: "Careful with rotation, if not put as default, SW axix swap is needed. Right now placed upsidedown, hence this is adjusted in SW."
- note removed: "Display"
- note removed: "Display backlight"
- note removed: "Dock connector"
- note removed: "ESD protection"
- note removed: "GPIO"
- note removed: "Gas, Pressure, Temperature & Humidity"
- note removed: "High accuracy pressure sensor"
- note removed: "I2C addresses -------------------- BMI270 0x68 BMP581 0x46 BME688 0x76 LIS2MDLTR 0x1E APDS-9306-065 0x52"
- note removed: "IMU with step counter, gesture detection etc."
- note removed: "LiPo Charger"
- note removed: "Light sensor"
- note removed: "Magnetometer"
- note removed: "NTS0104GU12 has internal pullups. Works for I2C. https://www.nxp.com/docs/en/data-sheet/NTS0104.pdf"
- note removed: "Power Management"
- note removed: "Pull down all EN. Battery is connected directly to some of those ICs but since EN is pulled low and only set high by ANNA, they will be off when battery is low (NORA shut off)."
- note removed: "Pull-up/down resistors"
- note removed: "SELI LOW => charge with 100mA SELV HIGH => charge to 4.2V"
- note removed: "SWD pins will probably touch the skin, hence we need ESD protection. Those are not for 1.8V, but they will limit significatnly and then interna nRF chip ESD protection handles the rest(if I understand correctly)."
- note removed: "Test Points"
- note removed: "Vibration motor (ERM Mode)"
- moved on the sheet: M1A, M1B, M1C, X2

Commit message: Working on USB test board
Parts:
- added C10, C11, C6, C7, C9: 10u, Capacitor_SMD:C_0603_1608Metric, symbol Device:C_Small
- added C3, C5: 1u, Capacitor_SMD:C_0603_1608Metric, symbol Device:C_Small
- added C4: 2u2, Capacitor_SMD:C_0603_1608Metric, symbol Device:C_Small
- added C8: 100n, Capacitor_SMD:C_0603_1608Metric, symbol Device:C_Small
- added IC3: nPM1300-QEXX, Package_DFN_QFN:QFN-32-1EP_5x5mm_P0.5mm_EP3.6x3.6mm_ThermalVias, symbol Nordic:nPM1300-QEXX
- added L1, L2: 2u2, symbol Device:L
- added R10, R9: 1k8, Resistor_SMD:R_0603_1608Metric, symbol Device:R_Small
- added R11: 0R, Resistor_SMD:R_0603_1608Metric, symbol Device:R_Small
- added R12: 10k, Resistor_SMD:R_0603_1608Metric, symbol Device:R_Small
- added R7: 47k, Resistor_SMD:R_0603_1608Metric, symbol Device:R_Small
- added R8: 150k, Resistor_SMD:R_0603_1608Metric, symbol Device:R_Small
- added X3: VBUS, Connector_PinHeader_2.54mm:PinHeader_1x02_P2.54mm_Vertical, symbol Connector_Generic:Conn_01x02
- added X4: VBAT, Molex:78171-0002, symbol Connector_Generic:Conn_01x02
- added X5: INT, Connector_PinHeader_2.54mm:PinHeader_1x02_P2.54mm_Vertical, symbol Connector_Generic:Conn_01x02
- IC2: symbol NXP:NX3DV42 -> TexasInstruments_Kampi:TS3USB221A
- X1: value Conn_01x02 -> VDISPLAY
Connections:
- net +1V8: now also C6.1, C8.1, IC3.12 (VDDIO), IC3.3 (SW1), L1.2, R10.2, R12.2, R9.2; no longer X1.1 (Pin_1)
- net D+/SWDCLK: now also IC2.8 (D+); no longer IC2.1 (D+)
- net D-/SWDIO: now also IC2.7 (D-); no longer IC2.2 (D-)
- net GND: now also IC2.5 (GND), IC2.6 (~{OE}), X1.1 (Pin_1), C10.2, C11.2, C3.2, C4.2, C5.2, C6.2, C7.2, C8.2, C9.2, IC3.15 (SHPHLD), IC3.2 (PVSS1), IC3.33 (AVSS), IC3.6 (PVSS2), R11.1, R7.1, R8.1, X3.2 (Pin_2), X4.2 (Pin_2), X5.2 (Pin_2); no longer IC2.3 (GND), IC2.8 (~{OE}), X1.2 (Pin_2)
- net MCU_D+: now also IC2.3 (2D+); no longer IC2.7 (HSDI2+)
- net MCU_D-: now also IC2.4 (2D-); no longer IC2.6 (HSD2-)
- net MCU_SWDCLK: now also IC2.1 (1D+); no longer IC2.5 (HSDI1+)
- net MCU_SWDIO: now also IC2.2 (1D-); no longer IC2.4 (HSD1-)
- net SEL_SWD: now also IC2.9 (S); no longer IC2.10 (S)
- net VBUS: now also C3.1, IC3.21 (VBUS), X3.1 (Pin_1); no longer C2.1, IC2.9 (Vcc), M1.B9 (VBUS), R4.1
- new net: IC3.17 (VSET1), R7.2
- new net: IC3.7 (GPIO0), R12.1, X5.1 (Pin_1)
- new net: IC3.1 (VOUT1), L1.1
- new net: IC3.16 (VSET2), R8.2
- new net: IC3.18 (NTC), R11.2
- new net: C4.1, IC3.19 (VBAT), X4.1 (Pin_1)
- new net: C5.1, IC3.22 (VBUSOUT), M1.B9 (VBUS)
- new net: IC3.29 (LSOUT1/VOUTLDO1), X1.2 (Pin_2)
- new net: IC3.32 (VOUT2), L2.1
- new net +3V0: C2.1, C7.1, IC2.10 (VDD), IC3.5 (SW2), L2.2, R4.1
- new net SCL: IC3.14 (SCL), R10.1
- new net SDA: IC3.13 (SDA), R9.1
- new net VSYS: C10.1, C11.1, C9.1, IC3.20 (VSYS), IC3.28 (LSIN1/VINLDO1), IC3.4 (PVDD)
- no-connect marks 49 -> 60
Other:
- note removed: "External 16MB Flash"
- note removed: "Microcontroller (NORA-B106/nRF5340)"
- moved on the sheet: C1, IC1, M1A, M1B, M1C, R1, R2, R3, X2

Commit message: Working on nPM1300 design
Parts:
- removed R11: 0R, Resistor_SMD:R_0603_1608Metric, symbol Device:R_Small
- removed R12: 10k, Resistor_SMD:R_0603_1608Metric, symbol Device:R_Small
- C10, C11, C6, C7, C9: Distributor (none) -> Mouser; Mfr. (none) -> KYOCERA AVX; Mfr. No. (none) -> CM105X5R106M25AT; Order Number (none) -> 346-CM105X5R106M25AT
- IC2: value NX3DV42 -> TS3USB221A; footprint (none) -> Package_QFN:UQFN-10_1.55x2.05mm_P0.5mm; Distributor (none) -> Mouser; Mfr. (none) -> Texas Instruments; Mfr. No. (none) -> TS3USB221A; Order Number (none) -> 595-TS3USB221A
- L1, L2: footprint (none) -> Inductor_SMD_Kampi:L_0806_2016; Distributor (none) -> Mouser; Mfr. (none) -> Samsung Electro-Mechanics; Mfr. No. (none) -> CIGT201610EH2R2MNE; Order Number (none) -> 187-CIGT201610EH2R2M
- R7: value 47k -> 150k
- R8: value 150k -> 47k; now not fitted; now left out of the parts list
Connections:
- net +1V8: now also C7.1, IC3.32 (VOUT2), L2.1; no longer C6.1, IC3.3 (SW1), L1.2
- net +3V0: now also C6.1, IC3.1 (VOUT1), L1.1; no longer C7.1, IC3.5 (SW2), L2.2
- net GND: now also IC3.18 (NTC)
- net at X5.1 (Pin_1): now also IC3.11 (GPIO4); no longer IC3.7 (GPIO0)
- new net: IC3.5 (SW2), L2.2
- new net: IC3.3 (SW1), L1.2
Other:
- moved on the sheet: C10, C11, C6, C7, C9, L1

Commit message: Working on nPM1300 design
Connections:
- net MCU-D+ renamed MCU_D_N
- net MCU_D_N: now also IC2.4 (2D-)
- net MCU_D+ renamed MCU_D_P
- net MCU_D_P: now also M1.D9 (D-)
- removed net MCU_D-: IC2.4 (2D-), M1.D9 (D-)
- net MCU_RESETn: no longer names the net of M1.J3 (~{RESET})
- no-connect marks 60 -> 61
Changed lines of the file:
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@@
   (no_connect (at 367.03 154.94))
   (no_connect (at 55.88 151.13))
+  (no_connect (at 209.55 162.56))
   (no_connect (at 306.07 106.68))
   (no_connect (at 306.07 132.08))
@@
     (stroke (width 0) (type default))
   )
-  (wire (pts (xy 207.01 162.56) (xy 209.55 162.56))
-    (stroke (width 0) (type default))
-  )
   (wire (pts (xy 143.51 170.18) (xy 143.51 171.45))
     (stroke (width 0) (type default))
@@
     (effects (font (size 1.27 1.27)) (justify left bottom))
   )
-  (global_label "MCU_RESETn" (shape input) (at 207.01 162.56 180) (fields_autoplaced)
-    (effects (font (size 1.27 1.27)) (justify right))
-    (property "Intersheetrefs" "${INTERSHEET_REFS}" (at 192.1906 162.56 0)
-      (effects (font (size 1.27 1.27)) (justify right) hide)
-    )
-  )
   (global_label "SEL_SWD" (shape output) (at 27.94 21.59 0) (fields_autoplaced)
     (effects (font (size 1.27 1.27)) (justify left))
@@
     )
   )
-  (global_label "MCU_D-" (shape bidirectional) (at 137.16 52.07 0) (fields_autoplaced)
-    (effects (font (size 1.27 1.27)) (justify left))
-    (property "Intersheetrefs" "${INTERSHEET_REFS}" (at 149.039 52.07 0)
+  (global_label "MCU_D_N" (shape bidirectional) (at 137.16 52.07 0) (fields_autoplaced)
+    (effects (font (size 1.27 1.27)) (justify left))
+    (property "Intersheetrefs" "${INTERSHEET_REFS}" (at 149.7647 52.07 0)
       (effects (font (size 1.27 1.27)) (justify left) hide)
     )
@@
     )
   )
-  (global_label "MCU_D+" (shape bidirectional) (at 137.16 54.61 0) (fields_autoplaced)
-    (effects (font (size 1.27 1.27)) (justify left))
-    (property "Intersheetrefs" "${INTERSHEET_REFS}" (at 149.039 54.61 0)
+  (global_label "MCU_D_P" (shape bidirectional) (at 137.16 54.61 0) (fields_autoplaced)
+    (effects (font (size 1.27 1.27)) (justify left))
+    (property "Intersheetrefs" "${INTERSHEET_REFS}" (at 149.7042 54.61 0)
       (effects (font (size 1.27 1.27)) (justify left) hide)
     )
@@
     )
   )
-  (global_label "MCU_D-" (shape bidirectional) (at 207.01 152.4 180) (fields_autoplaced)
-    (effects (font (size 1.27 1.27)) (justify right))
-    (property "Intersheetrefs" "${INTERSHEET_REFS}" (at 195.131 152.4 0)
+  (global_label "MCU_D_P" (shape bidirectional) (at 207.01 152.4 180) (fields_autoplaced)
+    (effects (font (size 1.27 1.27)) (justify right))
+    (property "Intersheetrefs" "${INTERSHEET_REFS}" (at 194.4658 152.4 0)
       (effects (font (size 1.27 1.27)) (justify right) hide)
     )
@@
     )
   )
-  (global_label "MCU-D+" (shape bidirectional) (at 207.01 154.94 180) (fields_autoplaced)
-    (effects (font (size 1.27 1.27)) (justify right))
-    (property "Intersheetrefs" "${INTERSHEET_REFS}" (at 194.5262 154.94 0)
-      (effects (font (size 1.27 1.27)) (justify right) hide)
-    )
+  (global_label "MCU_D_N" (shape bidirectional) (at 207.01 154.94 180) (fields_autoplaced)
+    (effects (font (size 1.27 1.27)) (justify right))
+    (property "Intersheetrefs" "${INTERSHEET_REFS}" (at 194.4053 154.94 0)
+      (effects (font (size 1.27 1.27)) (justify right) hide)
+    )

Commit message: First design for PCBWay
Parts:
- removed R4: 100k, Resistor_SMD:R_0603_1608Metric, symbol Device:R_Small
- added R8: 0R, Resistor_SMD:R_0805_2012Metric_Pad1.20x1.40mm_HandSolder, symbol Device:R_Small
- added S1: TL6340AF160Q, E-Switch:TL6340AF160Q_Modified, symbol Switch:SW_Push
- added TP1: 3V3, TestPoint:TestPoint_Pad_1.0x1.0mm, symbol Connector:TestPoint
- added TP2: 3V0, TestPoint:TestPoint_Pad_1.0x1.0mm, symbol Connector:TestPoint
- added TP3: 1V8, TestPoint:TestPoint_Pad_1.0x1.0mm, symbol Connector:TestPoint
- added TP4: GND, TestPoint:TestPoint_Pad_1.0x1.0mm, symbol Connector:TestPoint
- C1: renamed from C4; Distributor (none) -> Mouser; Mfr. (none) -> KYOCERA AVX; Mfr. No. (none) -> 06036D225KAT2A; Order Number (none) -> 581-06036D225KAT2A
- C10: renamed from C5; Distributor (none) -> Mouser; Mfr. (none) -> KYOCERA AVX; Mfr. No. (none) -> 0603YC105JAT2A; Order Number (none) -> 581-0603YC105JAT2A
- C2: renamed from C3; Distributor (none) -> Mouser; Mfr. (none) -> KYOCERA AVX; Mfr. No. (none) -> 0603YC105JAT2A; Order Number (none) -> 581-0603YC105JAT2A
- IC1: renamed from IC3; Distributor (none) -> Mouser; Mfr. (none) -> Nordic Semiconductor; Mfr. No. (none) -> nPM1300-QEAA-R7; Order Number (none) -> 949-NPM1300-QEAA-R7
- IC3: renamed from IC1; Mfr. Renesas -> GigaDevice; Mfr. No. AT25SL128A-MHE-T -> GD25LE255EWIGR; Order Number 988-AT25SL128A-MHE-T -> 363-GD25LE255EWIGR
- R1: renamed from R10; Distributor (none) -> Mouser; Mfr. (none) -> Vishay / Dale; Mfr. No. (none) -> CRCW060311K8FKEA; Order Number (none) -> 71-CRCW0603-11.8K-E3
- R2: renamed from R9; Distributor (none) -> Mouser; Mfr. (none) -> Vishay / Dale; Mfr. No. (none) -> CRCW060311K8FKEA; Order Number (none) -> 71-CRCW0603-11.8K-E3
- R3: renamed from R7; Distributor (none) -> Mouser; Mfr. (none) -> YAGEO; Mfr. No. (none) -> RC0603FR-07150KL; Order Number (none) -> 603-RC0603FR-07150KL
- R4: renamed from R8; Distributor (none) -> Mouser; Mfr. (none) -> YAGEO; Mfr. No. (none) -> RC0603FR-0747KL; Order Number (none) -> 603-RC0603FR-0747KL
- X5: renamed from X1; value VDISPLAY -> 3V3
- renumbered C1 to C11, C8 to C3, C2 to C4, C9 to C5, C7 to C6, C10 to C7, C6 to C8, C11 to C9, L2 to L1, L1 to L2, R1 to R5, R2 to R6, R3 to R7, X2 to X1, X5 to X2, X4 to X3, X3 to X4
Connections:
- net +1V8: now also TP3.1
- net +3V0: now also TP2.1
- net GND: now also X5.2 (Pin_2), S1.1, TP4.1; no longer IC1.15 (SHPHLD), X5.1 (Pin_1)
- net MCU_D_N: now also M1.D9 (D-); no longer M1.C9 (D+)
- net MCU_D_P: now also M1.C9 (D+); no longer M1.D9 (D-)
- net SCL: now also M1.E1 (P0.18/QSPI_CS)
- net SDA: now also M1.F1 (P0.17/QSPI_CLK)
- net BTN: now reaches M1.H8 (P0.30)
- net BTN: now also IC1.15 (SHPHLD), S1.2
- net INT: now reaches M1.J9 (P0.31)
- net INT: now also IC1.11 (GPIO4), X2.1 (Pin_1)
- net at C1.1, X3.1 (Pin_1): now also R8.2; no longer IC1.19 (VBAT)
- net at IC1.29 (LSOUT1/VOUTLDO1): now also X5.1 (Pin_1), TP1.1; no longer X5.2 (Pin_2)
- new net: IC1.19 (VBAT), R8.1
- no-connect marks 61 -> 57
Other:
- moved on the sheet: R3, R4, X5
