File: project/ZSWatch.kicad_pcb (KiCad board)
At the start: 4 copper layers, 41 x 38 mm, 35 parts, among them IC1 nPM1300-QEXX, IC2 TS3USB221A, IC3 AT25SL128A, M1 NORA-B106, X1 DOCK, X2 INT, X3 VBAT, X4 VBUS, X5 SEL, X6 3V3

Commit message: Working on nPM circuit
Parts:
- R1: value 150k -> 47k
- R2: value 47k -> 150k
Connections:
- TP3 pad 1: +3V0 -> +1V8
- TP4 pad 1: +1V8 -> +3V0
Routing:
- net +3V0: track 65.1 -> 65.7 mm
Changed lines of the file:
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@@
   (title_block
     (title "ZSWatch v2")
-    (date "2023-08-19")
+    (date "2023-10-26")
     (rev "3")
     (company "github.com/jakkra/ZSWatch-HW")
@@
       (stroke (width 0.05) (type solid)) (layer "F.CrtYd"))
     (pad "1" smd rect (at 0 0) (size 1 1) (layers "F.Cu" "F.Mask")
-      (net 6 "+3V0") (pinfunction "1") (pintype "passive"))
+      (net 3 "+1V8") (pinfunction "1") (pintype "passive"))
   )
   (footprint "Capacitor_SMD:C_0603_1608Metric" (layer "F.Cu")
@@
       (stroke (width 0.05) (type solid)) (layer "F.CrtYd"))
     (pad "1" smd rect (at 0 0) (size 1 1) (layers "F.Cu" "F.Mask")
-      (net 3 "+1V8") (pinfunction "1") (pintype "passive"))
+      (net 6 "+3V0") (pinfunction "1") (pintype "passive"))
   )
   (footprint "TestPoint:TestPoint_Pad_1.0x1.0mm" (layer "F.Cu")
@@
     (property "Distributor" "Mouser")
     (property "Mfr." "YAGEO")
-    (property "Mfr. No." "RC0603FR-0747KL")
-    (property "Order Number" "603-RC0603FR-0747KL")
+    (property "Mfr. No." "")
+    (property "Order Number" "")
     (property "Sheetfile" "ZSWatch.kicad_sch")
     (property "Sheetname" "")
-    (property "dnp" "")
-    (property "exclude_from_bom" "")
     (property "ki_description" "Resistor, small symbol")
     (property "ki_keywords" "R resistor")
-    (attr smd exclude_from_bom)
+    (attr smd)
     (fp_text reference "R2" (at 0 -1.43 90) (layer "F.SilkS") hide
         (effects (font (size 1 1) (thickness 0.15)))
     )
-    (fp_text value "47k" (at 0 1.43 90) (layer "F.Fab") hide
+    (fp_text value "150k" (at 0 1.43 90) (layer "F.Fab") hide
         (effects (font (size 1 1) (thickness 0.15)))
     )
@@
     (property "Distributor" "Mouser")
     (property "Mfr." "YAGEO")
-    (property "Mfr. No." "RC0603FR-07150KL")
-    (property "Order Number" "603-RC0603FR-07150KL")
+    (property "Mfr. No." "")
+    (property "Order Number" "")
     (property "Sheetfile" "ZSWatch.kicad_sch")
     (property "Sheetname" "")
@@
         (effects (font (size 1 1) (thickness 0.15)))
     )
-    (fp_text value "150k" (at 0 1.43) (layer "F.Fab") hide
+    (fp_text value "47k" (at 0 1.43) (layer "F.Fab") hide
         (effects (font (size 1 1) (thickness 0.15)))
     )
@@
     (tags "resistor")
     (property "Distributor" "Mouser")
-    (property "Mfr." "Vishay / Dale")
-    (property "Mfr. No." "CRCW060311K8FKEA")
-    (property "Order Number" "71-CRCW0603-11.8K-E3")
+    (property "Mfr." "")
+    (property "Mfr. No." "")
+    (property "Order Number" "")
     (property "Sheetfile" "ZSWatch.kicad_sch")
     (property "Sheetname" "")
@@
     (descr "Resistor SMD 0603 (1608 Metric), square (rectangular) end terminal, IPC_7351 nominal, (Body size source: IPC-SM-782 page 72, https://www.pcb-3d.com/wordpress/wp-content/uploads/ipc-sm-782a_amendment_1_and_2.pdf), generated with kicad-footprint-generator")
     (tags "resistor")
-    (property "Distributor" "Mouser")
-    (property "Mfr." "Vishay / Dale")
-    (property "Mfr. No." "CRCW060311K8FKEA")
-    (property "Order Number" "71-CRCW0603-11.8K-E3")
+    (property "Distributor" "")
+    (property "Mfr." "")
+    (property "Mfr. No." "")
+    (property "Order Number" "")
     (property "Sheetfile" "ZSWatch.kicad_sch")
     (property "Sheetname" "")
@@
   (segment (start 167.6686 109.397797) (end 167.6686 110.497798) (width 0.4) (layer "F.Cu") (net 3))
   (segment (start 159.512 110.109) (end 159.512 111.112) (width 0.4) (layer "F.Cu") (net 3))
+  (segment (start 145.034 115.5) (end 143.8 115.5) (width 0.4) (layer "F.Cu") (net 3))
   (segment (start 160.782 110.998) (end 160.668 111.112) (width 0.2) (layer "F.Cu") (net 3))
   (segment (start 171.75 120.176) (end 171.052 120.176) (width 0.2) (layer "F.Cu") (net 3))
@@
   (segment (start 159.697 97.234) (end 160.228 97.234) (width 0.3) (layer "F.Cu") (net 3))
   (segment (start 161.728 102.87) (end 161.728 103.632) (width 0.2) (layer "F.Cu") (net 3))
-  (segment (start 143.8 110.1) (end 143.8 111.1) (width 0.4) (layer "F.Cu") (net 3))
   (segment (start 166.671 120.176) (end 167.369 120.176) (width 0.2) (layer "F.Cu") (net 3))
   (segment (start 161.393 110.998) (end 160.782 110.998) (width 0.2) (layer "F.Cu") (net 3))
@@
   (via (at 167.369 120.176) (size 0.45) (drill 0.25) (layers "F.Cu" "B.Cu") (net 3))
   (via (at 161.728 102.87) (size 0.45) (drill 0.25) (layers "F.Cu" "B.Cu") (net 3))
-  (via (at 143.8 110.1) (size 0.8) (drill 0.4) (layers "F.Cu" "B.Cu") (net 3))
   (via (at 159.616 117.602) (size 0.45) (drill 0.25) (layers "F.Cu" "B.Cu") (net 3))
   (via (at 171.052 120.176) (size 0.45) (drill 0.25) (layers "F.Cu" "B.Cu") (net 3))
+  (via (at 145.034 115.5) (size 0.8) (drill 0.4) (layers "F.Cu" "B.Cu") (net 3))
   (segment (start 159.697 97.234) (end 159.695 97.232) (width 0.3) (layer "B.Cu") (net 3))
   (segment (start 156.444 97.232) (end 154.444 99.232) (width 0.3) (layer "B.Cu") (net 3))
@@
   (segment (start 164.602 118.3) (end 163.1 116.798) (width 0.2) (layer "In2.Cu") (net 5))
   (segment (start 171.543602 118.3) (end 164.602 118.3) (width 0.2) (layer "In2.Cu") (net 5))
-  (segment (start 148.3 115.5) (end 149.5 114.3) (width 0.4) (layer "F.Cu") (net 6))
+  (segment (start 148.763 111.1) (end 149.5 110.363) (width 0.4) (layer "F.Cu") (net 6))
+  (segment (start 155.216 97.117) (end 155.956 97.117) (width 0.4) (layer "F.Cu") (net 6))
+  (segment (start 153.533 98.8) (end 155.216 97.117) (width 0.4) (layer "F.Cu") (net 6))
   (segment (start 159.528 97.934) (end 159.247 97.653) (width 0.2) (layer "F.Cu") (net 6))
-  (segment (start 157.2 125.7) (end 152.3 125.7) (width 0.2) (layer "F.Cu") (net 6))
+  (segment (start 143.8 111.1) (end 148.763 111.1) (width 0.4) (layer "F.Cu") (net 6))
   (segment (start 165.862 106.374) (end 165.862 107.797) (width 0.2) (layer "F.Cu") (net 6))
-  (segment (start 153.533 98.8) (end 155.216 97.117) (width 0.4) (layer "F.Cu") (net 6))
+  (segment (start 152.3 125.7) (end 149.5 122.9) (width 0.2) (layer "F.Cu") (net 6))
   (segment (start 150.49 107.797) (end 149.5 106.807) (width 0.2) (layer "F.Cu") (net 6))
   (segment (start 149.5 106.807) (end 149.5 100.436) (width 0.4) (layer "F.Cu") (net 6))
-  (segment (start 149.4 116.6) (end 148.3 115.5) (width 0.2) (layer "F.Cu") (net 6))
-  (segment (start 143.8 115.5) (end 148.3 115.5) (width 0.4) (layer "F.Cu") (net 6))
-  (segment (start 149.4 122.8) (end 149.4 116.6) (width 0.2) (layer "F.Cu") (net 6))
-  (segment (start 149.5 114.3) (end 149.5 106.807) (width 0.4) (layer "F.Cu") (net 6))
+  (segment (start 149.5 110.363) (end 149.5 106.807) (width 0.4) (layer "F.Cu") (net 6))
+  (segment (start 149.5 122.9) (end 149.5 110.363) (width 0.2) (layer "F.Cu") (net 6))
+  (segment (start 157.2 125.7) (end 152.3 125.7) (width 0.2) (layer "F.Cu") (net 6))
   (segment (start 151.136 98.8) (end 153.533 98.8) (width 0.4) (layer "F.Cu") (net 6))
   (segment (start 159.247 95.782) (end 159.271 95.758) (width 0.2) (layer "F.Cu") (net 6))
   (segment (start 149.5 100.436) (end 151.136 98.8) (width 0.4) (layer "F.Cu") (net 6))
-  (segment (start 155.216 97.117) (end 155.956 97.117) (width 0.4) (layer "F.Cu") (net 6))
-  (segment (start 152.3 125.7) (end 149.4 122.8) (width 0.2) (layer "F.Cu") (net 6))
   (segment (start 159.247 97.653) (end 159.247 95.782) (width 0.2) (layer "F.Cu") (net 6))
   (segment (start 165.862 107.797) (end 150.49 107.797) (width 0.2) (layer "F.Cu") (net 6))

Commit message: Add missing output capacitor for LDO output
Parts:
- added C12: 10u, Capacitor_SMD:C_0603_1608Metric, F.Cu at (161.7, 95.6)
Connections:
- C4 pad 1: +3V0 -> +1V8
- C6 pad 1: +1V8 -> +3V0
- C8 pad 1: +3V0 -> +1V8
- IC1 pad 1: +3V0 -> +1V8
- IC1 pad 32: +1V8 -> +3V0
- IC2 pad 10: +3V0 -> +1V8
- L1 pad 1: +1V8 -> +3V0
- L2 pad 1: +3V0 -> +1V8
- TP3 pad 1: +1V8 -> +3V0
- TP4 pad 1: +3V0 -> +1V8
- X5 pad 1: +3V0 -> +1V8
Routing:
- net +3V0: track 65.7 -> 7.85 mm, vias 0 -> 3
- net +1V8: track 17.2 -> 75.0 mm, vias 9 -> 6
- net Net-(IC1-LSOUT1/VOUTLDO1): track 41.7 -> 43.2 mm
- net GND: track 35.3 -> 36.1 mm, vias 20 -> 21
