File: project/ZSWatch.kicad_pcb (KiCad board)
At the start: 4 copper layers, 41 x 38 mm, 86 parts, among them IC101 nPM1300-QEXX, IC201 APDS-9306-065, IC202 BMI270, IC203 BMP581, IC204 LIS2MDLTR, IC205 BME688, IC301 ESDALC6V1W5, IC302 FAN5622SX, IC303 MX25L51245GZ2I, IC304 TS3USB221A, IC305 NTS0104GU12, IC306 DRV2603RUNT, IC307 RV-8263-C8, M301 NORA-B106, Q201 DMG1013UW-7, Q301 BC817W, X101 BATTERY, X301 DOCK, X302 GC9A01A_CST816S, X303 M+, X304 M-

Commit message: Fix different manufacturing issues
Other:
- board text added: "0,196 mm"
- board text added: "0,43 mm"
- board text added: "Blue"
- board text removed: "0,11 mm"
- board text removed: "0,6 mm"
