File: project/MCU.kicad_sch (KiCad schematic)
At the start: 40 parts, among them IC301 ESDALC6V1W5, IC302 FAN5622SX, IC303 MX25U51245GZ4I00, IC304 TS3USB221A, IC305 NTS0104GU12, IC306 DRV2603RUNT, IC307 RV-8263-C8, M301 NORA-B106, M302 Vibrator DC Motor, Q301 BC817W, X301 DOCK, X302 GC9A01A_CST816S, X303 M+, X304 M-

Commit message: Fix different manufacturing issues
Parts:
- R305: now left out of the parts list
- R306: Mfr. No. CR0603-J/-000ELF -> CR0402-J/-000GLF; now not fitted
- R310: Mfr. No. CR0603-J/-000ELF -> CR0402-J/-000GLF
Other:
- note added: "NOTE: You can disable USB permanently by removing the voltage divider, bridge SWD by closing the jumper fields and assemble the resistor on the RESETn line. The voltage switch should only be active when a dock is connected and the switch need ~30 uA of current so we can not use a Z-Diode for the power supply. Voltage stability doesn´t care because the IC can work from 2.3 to 5.5 V. We set the "no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"
- note removed: "NOTE: You can disable USB permanently by removing the voltage divider and bridge SWD by closing the jumper fields. The voltage switch should only be active when a dock is connected and the switch need ~30 uA of current so we can not use a Z-Diode for the power supply. Voltage stability doesn´t care because the IC can work from 2.3 to 5.5 V. We set the "normal" voltage to 3.6 V to add a bit safety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"
Changed lines of the file:
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@@
     (effects (font (size 1.27 1.27)) (justify left bottom))
   )
-  (text "NOTE: You can disable USB permanently by removing the voltage divider and bridge SWD\nby closing the jumper fields.\nThe voltage switch should only be active when a dock is connected and \nthe switch need ~30 uA of current so we can not use a Z-Diode for the power supply.\nVoltage stability doesn´t care because the IC can work from 2.3 to 5.5 V. We set the\n\"normal\" voltage to 3.6 V to add a bit safety against voltage drops.\n"
+  (text "NOTE: You can disable USB permanently by removing the voltage divider, bridge SWD\nby closing the jumper fields and assemble the resistor on the RESETn line.\nThe voltage switch should only be active when a dock is connected and \nthe switch need ~30 uA of current so we can not use a Z-Diode for the power supply.\nVoltage stability doesn´t care because the IC can work from 2.3 to 5.5 V. We set the\n\"normal\" voltage to 3.6 V to add a bit safety against voltage drops.\n"
     (at 160.02 283.21 0)
     (effects (font (size 1.27 1.27)) (justify left bottom))
@@
       (effects (font (size 1.27 1.27)) hide)
     )
-    (property "Mfr. No." "CR0603-J/-000ELF" (at 219.71 248.92 0)
+    (property "Mfr. No." "CR0402-J/-000GLF" (at 219.71 248.92 0)
       (effects (font (size 1.27 1.27)) hide)
     )
@@
   )
   (symbol (lib_id "Device:R_Small") (at 195.58 236.22 0) (mirror x) (unit 1)
-    (in_bom no) (on_board yes) (dnp no) (fields_autoplaced)
+    (in_bom no) (on_board yes) (dnp yes) (fields_autoplaced)
     (property "Reference" "R306" (at 193.04 234.95 0)
       (effects (font (size 1.27 1.27)) (justify right))
@@
       (effects (font (size 1.27 1.27)) hide)
     )
-    (property "Mfr. No." "CR0603-J/-000ELF" (at 195.58 236.22 0)
+    (property "Mfr. No." "CR0402-J/-000GLF" (at 195.58 236.22 0)
       (effects (font (size 1.27 1.27)) hide)
     )
@@
   )
   (symbol (lib_id "Device:R_Small") (at 185.42 236.22 0) (unit 1)
-    (in_bom yes) (on_board yes) (dnp yes) (fields_autoplaced)
+    (in_bom no) (on_board yes) (dnp yes) (fields_autoplaced)
     (property "Reference" "R305" (at 182.88 234.95 0)
       (effects (font (size 1.27 1.27)) (justify right))
