File: project/Power.kicad_sch (KiCad schematic)
At the start: 20 parts, among them IC101 nPM1300-QEXX, X101 BATTERY

Commit message: Fix different manufacturing issues
Parts:
- R103: Mfr. No. CR0603-J/-000ELF -> CR0402-J/-000GLF
Changed lines of the file:
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@@
       (effects (font (size 1.27 1.27)) hide)
     )
-    (property "Mfr. No." "CR0603-J/-000ELF" (at 135.89 63.5 0)
+    (property "Mfr. No." "CR0402-J/-000GLF" (at 135.89 63.5 0)
       (effects (font (size 1.27 1.27)) hide)
     )
